Commit message: description du robot urdf

File: crabe_description/urdf/crabebot.urdf (robot description, URDF)
Before this commit: robot crabe, 10 links, 9 joints
Links:
- removed link aileron
- removed link base
- removed link benne1
- removed link benne2
- removed link benne3
- removed link roue_droite
- removed link roue_gauche
- added link L_wheel, mass ${m_wheel}; collision cylinder length=${h_wheel} radius=${r_wheel}; visual cylinder length=${h_wheel} radius=${r_wheel}
- added link Left_arm, mass ${m_arm}; collision box size=${l_arm} ${L_arm} ${h_arm}; visual box size=${l_arm} ${L_arm} ${h_arm}
- added link R_wheel, mass ${m_wheel}; collision cylinder length=${h_wheel} radius=${r_wheel}; visual cylinder length=${h_wheel} radius=${r_wheel}
- added link Right_arm, mass ${m_arm}; collision box size=${l_arm} ${L_arm} ${h_arm}; visual box size=${l_arm} ${L_arm} ${h_arm}
- added link body, mass ${m_body}; collision box size=${l_body} ${L_body} ${h_body}; visual box size=${l_body} ${L_body} ${h_body}
Joints:
- removed joint base_to_aileron
- removed joint base_to_benne1
- removed joint base_to_cible_rouge
- removed joint base_to_cible_verte
- removed joint base_to_roue_droite
- removed joint base_to_roue_gauche
- removed joint benne_1_2
- removed joint benne_1_3
- removed joint benne_free_wheel
- added joint Body_L_wheel: type continuous, parent body, child L_wheel, origin xyz=0.1 ${L_body/2+eps_wheel} ${-h_body/2}, axis 0 1 0
- added joint Body_R_wheel: type continuous, parent body, child R_wheel, origin xyz=0.1 -${L_body/2+eps_wheel} ${-h_body/2}, axis 0 1 0
- added joint base_casterWheel: type fixed, parent body, child caster_wheel, origin xyz=-0.1 0 -${h_body/2 + free_r}
- added joint body_L_arm: type fixed, parent body, child Left_arm, origin xyz=${l_body/2 + l_arm/2} ${L_body/2+0.05} 0.1
- added joint body_R_arm: type fixed, parent body, child Right_arm, origin xyz=${l_body/2 + l_arm/2} -${L_body/2+0.05} 0.1
- added joint body_cible_rouge: type fixed, parent body, child cible_rouge, origin xyz=-0.15 -0.1 0.005
- added joint body_cible_verte: type fixed, parent body, child cible_verte, origin xyz=-0.15 0.1 0.005

Commit message: urdf fini

File: crabe_description/urdf/crabebot.urdf (robot description, URDF)
Before this commit: robot crabe, 8 links, 7 joints
Joints:
- joint base_casterWheel: origin xyz=-0.1 0 -${h_body/2 + free_r} -> xyz=-0.15 0 -${free_r + h_body/2}
- joint body_L_arm: origin xyz=${l_body/2 + l_arm/2} ${L_body/2+0.05} 0.1 -> xyz=${l_body/2} ${L_body/2*cos(alpha_arm)} -0.09 rpy=0 0 ${alpha_arm}
- joint body_R_arm: origin xyz=${l_body/2 + l_arm/2} -${L_body/2+0.05} 0.1 -> xyz=${l_body/2} -${L_body/2*cos(alpha_arm)} -0.09 rpy=0 0 -${alpha_arm}
- joint body_cible_rouge: origin xyz=-0.15 -0.1 0.005 -> xyz=-0.15 -0.1 ${h_body/2}
- joint body_cible_verte: origin xyz=-0.15 0.1 0.005 -> xyz=-0.15 0.1 ${h_body/2}

Commit message: ajout d'une mise à l'echelle du robot

File: crabe_description/urdf/crabebot.urdf (robot description, URDF)
Before this commit: robot crabe, 8 links, 7 joints
Links:
- link caster_wheel: mass ${free_m} -> ${m_free}; geometry collision sphere radius=${r_free}; visual sphere radius=${r_free}
Joints:
- joint Body_L_wheel: origin xyz=0.1 ${L_body/2+eps_wheel} ${-h_body/2} -> xyz=${l_body/4} ${L_body/2+h_wheel/2+eps_wheel} ${-h_body/2}
- joint Body_R_wheel: origin xyz=0.1 -${L_body/2+eps_wheel} ${-h_body/2} -> xyz=${l_body/4} -${L_body/2+h_wheel/2+eps_wheel} ${-h_body/2}
- joint base_casterWheel: origin xyz=-0.15 0 -${free_r + h_body/2} -> xyz=-${3*l_body/8} 0 -${r_free + h_body/2}
- joint body_L_arm: origin xyz=${l_body/2} ${L_body/2*cos(alpha_arm)} -0.09 rpy=0 0 ${alpha_arm} -> xyz=${l_body/2} ${L_body/2*cos(alpha_arm)} -${h_body/2+h_arm/2-0.01} rpy=0 0 ${alpha_arm}
- joint body_R_arm: origin xyz=${l_body/2} -${L_body/2*cos(alpha_arm)} -0.09 rpy=0 0 -${alpha_arm} -> xyz=${l_body/2} -${L_body/2*cos(alpha_arm)} -${h_body/2+h_arm/2-0.01} rpy=0 0 -${alpha_arm}
- joint body_cible_rouge: origin xyz=-0.15 -0.1 ${h_body/2} -> xyz=-${3*l_body/8} -${L_body/3} ${h_body/2}
- joint body_cible_verte: origin xyz=-0.15 0.1 ${h_body/2} -> xyz=-${3*l_body/8} ${L_body/3} ${h_body/2}

File: crabe_description/urdf/crabebot_test.urdf (robot description, URDF)
Before this commit: robot crabe, 8 links, 7 joints
Links:
- link Left_arm: geometry collision box size=0.3 0.3 0.1; visual box size=0.3 0.3 0.1
- link Right_arm: geometry collision box size=0.3 0.3 0.1; visual box size=0.3 0.3 0.1
Joints:
- joint base_casterWheel: origin xyz=-0.1 0 -0.1 -> xyz=-0.15000000000000002 0 -0.1
- joint body_L_arm: origin xyz=0.35 0.2 0.1 -> xyz=0.2 0.10606601717798213 -0.11 rpy=0 0 0.7853981633974483
- joint body_R_arm: origin xyz=0.35 -0.2 0.1 -> xyz=0.2 -0.10606601717798213 -0.11 rpy=0 0 -0.7853981633974483
- joint body_cible_rouge: origin xyz=-0.15 -0.1 0.005 -> xyz=-0.15000000000000002 -0.15 0.05
- joint body_cible_verte: origin xyz=-0.15 0.1 0.005 -> xyz=-0.15000000000000002 0.15 0.05

Commit message: modif arm angle

File: crabe_description/urdf/crabebot.urdf (robot description, URDF)
Before this commit: robot crabe, 8 links, 7 joints
Joints:
- joint body_L_arm: origin xyz=${l_body/2} ${L_body/2*cos(alpha_arm)} -${h_body/2+h_arm/2-0.01} rpy=0 0 ${alpha_arm} -> xyz=${cos(alpha_arm)*l_arm/2} ${sin(alpha_arm)*l_arm/2} -${h_body/2+h_arm/2} rpy=0 0 ${alpha_arm}
- joint body_R_arm: origin xyz=${l_body/2} -${L_body/2*cos(alpha_arm)} -${h_body/2+h_arm/2-0.01} rpy=0 0 -${alpha_arm} -> xyz=${cos(alpha_arm)*l_arm/2} -${sin(alpha_arm)*l_arm/2} -${h_body/2+h_arm/2} rpy=0 0 -${alpha_arm}

Commit message: ajout reservoir

File: crabe_description/urdf/crabebot.urdf (robot description, URDF)
Before this commit: robot crabe, 8 links, 7 joints
Links:
- removed link caster_wheel
- added link Left_mur, mass ${m_mur_long}; collision box size=${l_murs} ${e_murs} ${h_murs}; visual box size=${l_murs} ${e_murs} ${h_murs}
- added link Mur_f, mass ${m_mur_f}; collision box size=${l_mur_f} ${e_murs} ${h_murs}; visual box size=${l_mur_f} ${e_murs} ${h_murs}
- added link Right_mur, mass ${m_mur_long}; collision box size=${l_murs} ${e_murs} ${h_murs}; visual box size=${l_murs} ${e_murs} ${h_murs}
- added link caster_wheel_1, mass ${m_free}; collision sphere radius=${r_free}; visual sphere radius=${r_free}
- added link caster_wheel_2, mass ${m_free}; collision sphere radius=${r_free}; visual sphere radius=${r_free}
Joints:
- removed joint base_casterWheel
- added joint base_casterWheel_1: type fixed, parent body, child caster_wheel_1, origin xyz=-${3*l_body/8} ${3*L_body/8} -${r_free + h_body/2}
- added joint base_casterWheel_2: type fixed, parent body, child caster_wheel_2, origin xyz=-${3*l_body/8} -${3*L_body/8} -${r_free + h_body/2}
- added joint body_L_mur: type fixed, parent body, child Left_mur, origin xyz=0 ${l_mur_f/2 - e_murs/2} -${h_body/2+h_murs/2} rpy=0 0 0
- added joint body_R_mur: type fixed, parent body, child Right_mur, origin xyz=0 -${l_mur_f/2 - e_murs/2} -${h_body/2+h_murs/2} rpy=0 0 0
- added joint body_mur_f: type fixed, parent body, child Mur_f, origin xyz=-${l_body/2 + e_murs/2} 0 -${h_body/2+h_murs/2} rpy=0 0 ${pi/2}
- joint body_L_arm: origin xyz=${cos(alpha_arm)*l_arm/2} ${sin(alpha_arm)*l_arm/2} -${h_body/2+h_arm/2} rpy=0 0 ${alpha_arm} -> xyz=${cos(alpha_arm)*l_arm/2 + l_body/2} ${sin(alpha_arm)*l_arm/2 + l_mur_f/2 - e_murs/2} -${h_body/2+h_arm/2} rpy=0 0 ${alpha_arm}
- joint body_R_arm: origin xyz=${cos(alpha_arm)*l_arm/2} -${sin(alpha_arm)*l_arm/2} -${h_body/2+h_arm/2} rpy=0 0 -${alpha_arm} -> xyz=${cos(alpha_arm)*l_arm/2 + l_body/2} -${sin(alpha_arm)*l_arm/2 + l_mur_f/2 - e_murs/2} -${h_body/2+h_arm/2} rpy=0 0 -${alpha_arm}

Commit message: ajout des portes et des forces

File: crabe_description/urdf/crabebot.urdf (robot description, URDF)
Before this commit: robot crabe, 12 links, 11 joints
Links:
- added link Front_door, mass ${m_mur_f}; collision box size=${l_mur_f - 2*e_murs} ${e_murs} ${h_murs}; visual box size=${l_mur_f - 2*e_murs} ${e_murs} ${h_murs}
Joints:
- added joint body_front_door: type prismatic, parent body, child Front_door, origin xyz=${l_body/2 + e_murs/2} 0 -${h_body/2+h_murs/2} rpy=0 0 ${pi/2}, axis 0 0 1, limit lower=0 upper=${h_murs} effort=2000 velocity=10
- joint body_mur_f: axis (none) -> 0 0 1; limit (none) -> lower=0 upper=${h_murs} effort=2000 velocity=10; type fixed -> prismatic

Commit message: Image calibration

File: crabe_description/urdf/crabebot.urdf (robot description, URDF)
Before this commit: robot crabe, 12 links, 11 joints
Joints:
- joint body_cible_rouge: origin xyz=-${3*l_body/8} -${L_body/3} ${h_body/2} -> xyz=0 -${L_body/3} ${h_body/2}
- joint body_cible_verte: origin xyz=-${3*l_body/8} ${L_body/3} ${h_body/2} -> xyz=0 ${L_body/3} ${h_body/2}

Commit message: urdf fix

File: crabe_description/urdf/crabebot.urdf (robot description, URDF)
Before this commit: robot crabe, 13 links, 11 joints
Joints:
- added joint body_front_door: type prismatic, parent body, child Front_door, origin xyz=${l_body/2 + e_murs/2} 0 -${h_body/2+h_murs/2} rpy=0 0 ${pi/2}, axis 0 0 1, limit lower=0 upper=${h_murs} effort=2000 velocity=10
